File: regulateur5V_1x1/regulateur5V_1x1.kicad_sch (KiCad schematic)
At the start: 3 parts, among them J1 Screw_Terminal_01x02, J2 Screw_Terminal_01x02, U1 LM7805_TO220

Commit message: MAJ
Parts:
- added C1: 220nF, symbol Device:C
- added C2, C4: 100nF, symbol Device:C
- added C3: 10uF, symbol Device:C
Connections:
- net GND: now also C1.2, C2.2, C3.2, C4.2
- net at J2.1 (Pin_1), U1.3 (VO): now also C3.1, C4.1
- net at J1.1 (Pin_1), U1.1 (VI): now also C1.1, C2.1

Commit message: hh
Parts:
- C1, C2, C4: footprint (none) -> Capacitor_THT:C_Disc_D5.0mm_W2.5mm_P5.00mm
- C3: footprint (none) -> Capacitor_THT:CP_Radial_D5.0mm_P2.00mm
Changed lines of the file:
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@@
 			)
 		)
-		(property "Footprint" ""
+		(property "Footprint" "Capacitor_THT:C_Disc_D5.0mm_W2.5mm_P5.00mm"
 			(at 157.1752 110.49 0)
 			(hide yes)
@@
 			)
 		)
-		(property "Footprint" ""
+		(property "Footprint" "Capacitor_THT:C_Disc_D5.0mm_W2.5mm_P5.00mm"
 			(at 87.3252 110.49 0)
 			(hide yes)
@@
 			)
 		)
-		(property "Footprint" ""
+		(property "Footprint" "Capacitor_THT:C_Disc_D5.0mm_W2.5mm_P5.00mm"
 			(at 70.8152 110.49 0)
 			(hide yes)
@@
 			)
 		)
-		(property "Footprint" ""
+		(property "Footprint" "Capacitor_THT:CP_Radial_D5.0mm_P2.00mm"
 			(at 138.1252 110.49 0)
 			(hide yes)
