File: regulateur5V_1x1/regulateur5V_1x1.kicad_pcb (KiCad board)
At the start: 2 copper layers, 3 parts, among them J1 Screw_Terminal_01x02, J2 Screw_Terminal_01x02, U1 LM7805_TO220

Commit message: MAJ
Parts:
- added C1: 220nF, Capacitor_THT:C_Disc_D5.0mm_W2.5mm_P5.00mm, F.Cu at (48.5, 77.0)
- added C2: 100nF, Capacitor_THT:C_Disc_D5.0mm_W2.5mm_P5.00mm, F.Cu at (60.0, 77.0)
- added C3: 10uF, Capacitor_THT:CP_Radial_D5.0mm_P2.00mm, F.Cu at (104.0, 75.0)
- added C4: 100nF, Capacitor_THT:C_Disc_D5.0mm_W2.5mm_P5.00mm, F.Cu at (122.0, 73.5)
- moved J1 74.5 mm to (24.8, 77.0), turned to 90 degrees
- moved J2 40.6 mm to (137.5, 73.5), turned to -90 degrees
- moved U1 40.3 mm to (84.0, 74.0)

Commit message: MAJ
Parts:
- moved U1 53.0 mm to (137.0, 74.5)
- moved C1 53.0 mm to (101.5, 77.5)
- moved C2 53.0 mm to (113.0, 77.5)
- moved C3 53.0 mm to (157.0, 75.5)
- moved C4 53.0 mm to (175.0, 74.0)
- moved J1 53.0 mm to (77.8, 77.5)
- moved J2 53.0 mm to (190.5, 74.0)
Routing:
- net Net-(J1-Pin_1): track 0.00 -> 60.5 mm
- net GND: track 0.00 -> 58.9 mm
- net Net-(J2-Pin_1): track 0.00 -> 53.2 mm
- added copper zone on F.Cu, net GND
Other:
- board outline added: 129.5 x 30 mm
- board text added: "BOSON-ENGINEERING"
